Commit message: Fixed deck heights and added IR sensors.

File: romeo-robot.urdf (robot description, URDF)
Before this commit: robot pi_robot, 5 links, 0 joints
Links:
- added link front_ir_sensor_link; visual box size=0.0445 0.0135 0.013
- added link left_front_ir_sensor_link; visual box size=0.0445 0.0135 0.013
- added link left_ir_sensor_link; visual box size=0.0445 0.0135 0.013
- added link right_front_ir_sensor_link; visual box size=0.0445 0.0135 0.013
- added link right_ir_sensor_link; visual box size=0.0445 0.0135 0.013
